File: hw/PowerExtractor.sch (EAGLE design)
At the start: 86 parts, among them IC1 LM358D, Q1 BSS84, Q2 IRL530, Q4 BC847SMD, Q7 IRF530, T1 IRL530N, T2 IRF7416, U1 ZXCT1086E5TA, U2 ZXCT1086E5TA

Commit message: Refactored PCB layout
Parts:
- D10: value 1N4148DO35-10 -> 1N4148MINIMELF; device triakcz:1N4148DO35-10 -> triakcz:1N4148MINIMELF
- R11, R4, R6: device rcl:R-EU_0207/10 -> rcl:R-EU_M0805
- renumbered DYNAMO to AC_IN
Connections:
- removed net N$36: D10.C, D12.C, KEYBOARD1.5
- new net N$41: A1.D4, D12.A
- net ARDUINO_VOUT_SENSE: now also A1.A7; no longer A1.A3
- net HUB1: now also R24.2; no longer R25.2
- net HUB2: now also R25.2; no longer R24.2
- net N$39: now also KEYBOARD1.5; no longer D12.A
- net N$6: now also D10.C, D12.C; no longer A1.D4
Other:
- moved on the sheet: D12
Changed lines of the file:
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@@
 <part name="B1" library="rectifier" deviceset="RB1A" device=""/>
 <part name="D4" library="diode" deviceset="1N5908" device="" value="SB360"/>
-<part name="R4" library="rcl" deviceset="R-EU_" device="0207/10" value="15k"/>
+<part name="R4" library="rcl" deviceset="R-EU_" device="M0805" value="15k"/>
 <part name="R5" library="rcl" deviceset="R-EU_" device="M0805" value="4k7"/>
 <part name="C7" library="rcl" deviceset="C-EU" device="C0805" value="10n"/>
-<part name="DYNAMO" library="con-wago-500" deviceset="W237-102" device=""/>
+<part name="AC_IN" library="con-wago-500" deviceset="W237-102" device=""/>
 <part name="C4" library="rcl" deviceset="C-EU" device="C0805" value="1uF/50V"/>
 <part name="R3" library="rcl" deviceset="R-EU_" device="M0805" value="100k"/>
-<part name="R6" library="rcl" deviceset="R-EU_" device="0207/10" value="10k"/>
+<part name="R6" library="rcl" deviceset="R-EU_" device="M0805" value="10k"/>
 <part name="D6" library="diode" deviceset="ZENER-DIODE" device="SOD80C" value="BZV55C15SMD"/>
 <part name="F1" library="fuse" deviceset="SHK20L" device="" value="F3.15A"/>
@@
 <part name="BAT" library="con-wago-500" deviceset="W237-102" device=""/>
 <part name="DIRECT_CHARGE" library="con-wago-500" deviceset="W237-102" device=""/>
-<part name="R11" library="rcl" deviceset="R-EU_" device="0207/10" value="100k"/>
+<part name="R11" library="rcl" deviceset="R-EU_" device="M0805" value="100k"/>
 <part name="R12" library="rcl" deviceset="R-EU_" device="0207/10" value="47k"/>
 <part name="R13" library="rcl" deviceset="R-EU_" device="M1206" value="0R01"/>
@@
 <part name="D2" library="triakcz" deviceset="1N4148" device="MINIMELF"/>
 <part name="R10" library="rcl" deviceset="R-EU_" device="R0805" value="330k"/>
-<part name="D10" library="triakcz" deviceset="1N4148" device="DO35-10" value="1N4148DO35-10"/>
+<part name="D10" library="triakcz" deviceset="1N4148" device="MINIMELF" value="1N4148MINIMELF"/>
 <part name="D12" library="triakcz" deviceset="1N4148" device="MINIMELF"/>
 </parts>
@@
 <instance part="R5" gate="G$1" x="274.32" y="25.4" rot="R90"/>
 <instance part="C7" gate="G$1" x="281.94" y="22.86" rot="R180"/>
-<instance part="DYNAMO" gate="-1" x="-132.08" y="43.18"/>
-<instance part="DYNAMO" gate="-2" x="-132.08" y="20.32"/>
+<instance part="AC_IN" gate="-1" x="-132.08" y="43.18"/>
+<instance part="AC_IN" gate="-2" x="-132.08" y="20.32"/>
 <instance part="C4" gate="G$1" x="175.26" y="35.56"/>
 <instance part="R3" gate="G$1" x="248.92" y="78.74" rot="R90"/>
@@
 <instance part="R10" gate="G$1" x="149.86" y="60.96" rot="R180"/>
 <instance part="D10" gate="G$1" x="213.36" y="165.1" rot="R90"/>
-<instance part="D12" gate="G$1" x="124.46" y="228.6" rot="R90"/>
+<instance part="D12" gate="G$1" x="116.84" y="259.08" rot="R90"/>
 </instances>
 <busses>
@@
 <pinref part="B1" gate="1" pin="AC2"/>
 <wire x1="-86.36" y1="30.48" x2="-88.9" y2="30.48" width="0.1524" layer="91"/>
-<pinref part="DYNAMO" gate="-1" pin="KL"/>
-<pinref part="R25" gate="G$1" pin="2"/>
-<wire x1="-55.88" y1="7.62" x2="-86.36" y2="7.62" width="0.1524" layer="91"/>
-<wire x1="-86.36" y1="30.48" x2="-86.36" y2="7.62" width="0.1524" layer="91"/>
+<pinref part="AC_IN" gate="-1" pin="KL"/>
+<pinref part="R24" gate="G$1" pin="2"/>
+<wire x1="-55.88" y1="15.24" x2="-86.36" y2="15.24" width="0.1524" layer="91"/>
+<wire x1="-86.36" y1="15.24" x2="-86.36" y2="30.48" width="0.1524" layer="91"/>
 <junction x="-86.36" y="30.48"/>
 </segment>
@@
 <label x="281.94" y="185.42" size="1.778" layer="95" rot="R270"/>
 <wire x1="281.94" y1="238.76" x2="63.5" y2="238.76" width="0.1524" layer="91"/>
-<wire x1="63.5" y1="238.76" x2="63.5" y2="200.66" width="0.1524" layer="91"/>
-<wire x1="63.5" y1="200.66" x2="73.66" y2="200.66" width="0.1524" layer="91"/>
-<pinref part="A1" gate="G$1" pin="A3"/>
+<wire x1="63.5" y1="238.76" x2="63.5" y2="190.5" width="0.1524" layer="91"/>
+<pinref part="A1" gate="G$1" pin="A7"/>
+<wire x1="63.5" y1="190.5" x2="73.66" y2="190.5" width="0.1524" layer="91"/>
 </segment>
 </net>
@@
 <wire x1="50.8" y1="195.58" x2="73.66" y2="195.58" width="0.1524" layer="91"/>
 <pinref part="A1" gate="G$1" pin="A5"/>
-</segment>
-</net>
-<net name="N$36" class="0">
-<segment>
-<pinref part="KEYBOARD1" gate="A" pin="5"/>
-<wire x1="124.46" y1="231.14" x2="124.46" y2="276.86" width="0.1524" layer="91"/>
-<wire x1="124.46" y1="276.86" x2="78.74" y2="276.86" width="0.1524" layer="91"/>
-<wire x1="78.74" y1="276.86" x2="78.74" y2="284.48" width="0.1524" layer="91"/>
-<pinref part="D10" gate="G$1" pin="C"/>
-<wire x1="213.36" y1="167.64" x2="213.36" y2="276.86" width="0.1524" layer="91"/>
-<wire x1="213.36" y1="276.86" x2="124.46" y2="276.86" width="0.1524" layer="91"/>
-<junction x="124.46" y="276.86"/>
-<pinref part="D12" gate="G$1" pin="C"/>
 </segment>
 </net>
@@
 </segment>
 </net>
-<net name="N$6" class="0">
-<segment>
-<pinref part="KEYBOARD1" gate="A" pin="2"/>
-<wire x1="71.12" y1="284.48" x2="71.12" y2="269.24" width="0.1524" layer="91"/>
-<wire x1="71.12" y1="269.24" x2="116.84" y2="269.24" width="0.1524" layer="91"/>
-<wire x1="116.84" y1="269.24" x2="116.84" y2="213.36" width="0.1524" layer="91"/>
-<wire x1="116.84" y1="213.36" x2="114.3" y2="213.36" width="0.1524" layer="91"/>
-<pinref part="A1" gate="G$1" pin="D4"/>
-</segment>
-</net>
 <net name="N$31" class="0">
 <segment>
@@
 </segment>
 </net>
-<net name="N$39" class="0">
-<segment>
-<pinref part="D12" gate="G$1" pin="A"/>
-<wire x1="124.46" y1="190.5" x2="124.46" y2="226.06" width="0.1524" layer="91"/>
-<wire x1="114.3" y1="190.5" x2="124.46" y2="190.5" width="0.1524" layer="91"/>
-<pinref part="A1" gate="G$1" pin="D12(MISO)"/>
-</segment>
-</net>
 <net name="HUB2" class="0">
 <segment>
-<pinref part="DYNAMO" gate="-2" pin="KL"/>
+<pinref part="AC_IN" gate="-2" pin="KL"/>
 <wire x1="-127" y1="20.32" x2="-104.14" y2="20.32" width="0.1524" layer="91"/>
 <wire x1="-104.14" y1="30.48" x2="-104.14" y2="20.32" width="0.1524" layer="91"/>
 <pinref part="B1" gate="1" pin="AC1"/>
 <wire x1="-99.06" y1="30.48" x2="-104.14" y2="30.48" width="0.1524" layer="91"/>
-<pinref part="R24" gate="G$1" pin="2"/>
-<wire x1="-104.14" y1="15.24" x2="-55.88" y2="15.24" width="0.1524" layer="91"/>
-<wire x1="-104.14" y1="20.32" x2="-104.14" y2="15.24" width="0.1524" layer="91"/>
 <junction x="-104.14" y="20.32"/>
-</segment>
-</net>
+<pinref part="R25" gate="G$1" pin="2"/>
+<wire x1="-55.88" y1="7.62" x2="-104.14" y2="7.62" width="0.1524" layer="91"/>
+<wire x1="-104.14" y1="7.62" x2="-104.14" y2="20.32" width="0.1524" layer="91"/>
+</segment>
+</net>
+<net name="N$41" class="0">
+<segment>
+<wire x1="116.84" y1="213.36" x2="114.3" y2="213.36" width="0.1524" layer="91"/>
+<pinref part="A1" gate="G$1" pin="D4"/>
+<pinref part="D12" gate="G$1" pin="A"/>
+<wire x1="116.84" y1="256.54" x2="116.84" y2="213.36" width="0.1524" layer="91"/>
+</segment>
+</net>
+<net name="N$6" class="0">
+<segment>
+<pinref part="D10" gate="G$1" pin="C"/>
+<wire x1="213.36" y1="167.64" x2="213.36" y2="269.24" width="0.1524" layer="91"/>
+<wire x1="213.36" y1="269.24" x2="116.84" y2="269.24" width="0.1524" layer="91"/>
+<pinref part="KEYBOARD1" gate="A" pin="2"/>
+<wire x1="71.12" y1="284.48" x2="71.12" y2="269.24" width="0.1524" layer="91"/>
+<wire x1="71.12" y1="269.24" x2="116.84" y2="269.24" width="0.1524" layer="91"/>
+<pinref part="D12" gate="G$1" pin="C"/>
+<wire x1="116.84" y1="261.62" x2="116.84" y2="269.24" width="0.1524" layer="91"/>
+<junction x="116.84" y="269.24"/>
+</segment>
+</net>
+<net name="N$39" class="0">
+<segment>
+<pinref part="KEYBOARD1" gate="A" pin="5"/>
+<wire x1="78.74" y1="276.86" x2="78.74" y2="284.48" width="0.1524" layer="91"/>
+<wire x1="78.74" y1="276.86" x2="124.46" y2="276.86" width="0.1524" layer="91"/>
+<wire x1="114.3" y1="190.5" x2="124.46" y2="190.5" width="0.1524" layer="91"/>
+<pinref part="A1" gate="G$1" pin="D12(MISO)"/>
+<wire x1="124.46" y1="276.86" x2="124.46" y2="190.5" width="0.1524" layer="91"/>
+</segment>
+</net>

Commit message: Updated library - arduino removed holes from dimension layer
Parts:
- removed R31: 10k, rcl:R-EU_M0805
- removed U$2, U$3: BCV47, triakcz:BCV47
- added Q3: BC847SMD, triakcz:BC847SMD
- added Q5: IRL530, transistor-power:IRF530
- added R27: 2k2, rcl:R-EU_0207/10
- B1: value (none) -> 1.5A
- C10: value 47uF/63V -> 100N; device rcl:CPOL-EUE5-8.5 -> rcl:C-EUC0805
- C11: value 47uF/50V -> 10n; device rcl:CPOL-EUE5-8.5 -> rcl:C-EUC0805
- C12, C7: value 10n -> 100N
- C13: value 100N -> 100n
- C14: value 1uF/50V -> 100n
- C4: value 1uF/50V -> 10n
- C5: value 100N -> 47uF/63V; device rcl:C-EUC0805 -> rcl:CPOL-EUE5-8.5
- C6: value 100n -> 1uF/50V
- C8: value 100n -> 47uF/50V; device rcl:C-EUC0805 -> rcl:CPOL-EUE5-8.5
- C9: value 100N -> 1uF/50V
- D10, D9: value 1N4148MINIMELF -> BZV55C15SMD; device triakcz:1N4148MINIMELF -> diode:ZENER-DIODESOD80C
- D3: value 1N6267A -> 1N4148MINIMELF; device diode:1N6267A -> triakcz:1N4148MINIMELF
- D4: value SB360 -> 1N4148MINIMELF; device diode:1N5908 -> triakcz:1N4148MINIMELF
- D5: value BZV55C15SMD -> SB360; device diode:ZENER-DIODESOD80C -> diode:1N5908
- D6: value BZV55C15SMD -> 1N6267A; device diode:ZENER-DIODESOD80C -> diode:1N6267A
- Q1: value BSS84 -> IRL530N; device triakcz:BSS84 -> transistor-power:IRF530
- Q2: value IRL530 -> BSS84; device transistor-power:IRF530 -> triakcz:BSS84
- Q4: value BC847SMD -> IRF7416; device triakcz:BC847SMD -> triakcz:IRF7416
- R12: value 47k -> 10k; device rcl:R-EU_0207/10 -> rcl:R-EU_M0805
- R14: value 0R01 -> 47k; device rcl:R-EU_M1206 -> rcl:R-EU_M0805
- R16: value 10k -> 100k
- R17: value 100k -> 10k; device rcl:R-EU_0207/10 -> rcl:R-EU_M0805
- R18: value 100k -> 15k
- R19: value 330k -> 4k7
- R2: value 33K -> 330K; device rcl:R-EU_R0805 -> rcl:R-EU_M0805
- R20: value 2k2 -> 100k
- R22: value 2k2 -> 10k; device rcl:R-EU_0207/10 -> rcl:R-EU_M0805
- R23: value 100k -> 0R01; device rcl:R-EU_R0805 -> rcl:R-EU_M1206
- R24: value 330K -> 10k
- R25: value 330K -> 330k
- R26: value 100k -> 220R; device rcl:R-EU_R0805 -> rcl:R-EU_M0805
- R28: value 10k -> 100k; device rcl:R-EU_R0805 -> rcl:R-EU_M0805
- R29: value 10k -> 2k2; device rcl:R-EU_M0805 -> rcl:R-EU_0207/10
- R3: value 100k -> 47k; device rcl:R-EU_M0805 -> rcl:R-EU_0207/10
- R30, R6: value 10k -> 100k; device rcl:R-EU_M0805 -> rcl:R-EU_R0805
- R4: value 15k -> 10k
- R5: value 4k7 -> 100k; device rcl:R-EU_M0805 -> rcl:R-EU_0207/10
- R7: value 220R -> 10k; device rcl:R-EU_M0805 -> rcl:R-EU_R0805
- R8: value 100k -> 330K; device rcl:R-EU_0207/10 -> rcl:R-EU_M0805
- R9: value 47k -> 33K; device rcl:R-EU_M0805 -> rcl:R-EU_R0805
- T1: value IRL530N -> BCV47; device transistor-power:IRF530 -> triakcz:BCV47
- T2: value IRF7416 -> BCV47; device triakcz:IRF7416 -> triakcz:BCV47
- renumbered 12VOUT to X7, BAT to X3, DIRECT_CHARGE to DC_IN, DISPLAY to DSPL, HEAD_LED to X5, KEYBOARD1 to KEYBRD, PHOTORESIST to JP1, Q7 to Q6, TAIL_LED to X6, U$1 to X4, U$4 to T3
Connections:
- net +5V: now also C7.2, R3.2, R4.2, R7.2; no longer C13.2, R12.2, R28.2, R29.2
- net ARDUINO_LIGHT_IN: now also R3.1; no longer R12.1
- net ARDUINO_MAIN_LIGHT_CTRL: now also R20.2; no longer R17.2
- net ARDUINO_OUT_CHARGE_OUTPUT_CONTROL: now also R29.2; no longer R22.2
- net ARDUINO_OUT_TAIL_LIGHT: now also R27.2; no longer R20.2
- net ARDUINO_PWM_OUT: now also Q1.G; no longer T1.G
- net ARDUINO_ROTATION_INT: now also R6.1, R7.1, T2.C; no longer R26.1, R28.1, U$2.C
- net ARDUINO_SELF_POWER_OUT: now also D7.A; no longer D2.A
- net ARDUINO_VIN: now also C3.1, Q2.S, R18.2; no longer C14.1, Q1.S, R4.2
- net ARDUINO_VIN_ANALOG: now also C4.2, R8.1, R9.2; no longer C12.2, R1.1, R2.2
- net ARDUINO_VOUT_SENSE: now also C11.2, R18.1, R19.2; no longer C7.2, R4.1, R5.2
- net BAT+: now also F2.1A, F2.1B; no longer F1.1A, F1.1B
- net BAT+FUSED: now also D9.C, F2.2A, F2.2B, Q2.D, R16.2, R22.1, R23.1; no longer D6.C, F1.2A, F1.2B, Q1.D, R14.1, R3.2, R30.1
- net GND: now also C11.1, C14.1, C3.2, C4.1, C8.-, C9.2, D6.A, Q1.S, Q3.E, Q5.S, R14.1, R19.1, R28.2, R30.2, T1.E, T2.E; no longer C11.-, C12.1, C13.1, C14.2, C4.2, C8.1, D3.A, Q2.S, Q4.E, R18.2, R2.1, R23.2, R5.1, T1.S, U$2.E, U$3.E
- net HUB1: now also R1.2; no longer R24.2
- net HUB2: now also R2.2; no longer R25.2
- net LIGHTVCC: now also C13.2, D10.C, Q4.S, R25.2; no longer C6.2, D5.C, R19.2, T2.S
- net N$1: now also C10.2, R12.2; no longer C5.2, R16.2
- net N$10: now also F1.1A, F1.1B; no longer F2.1A, F2.1B
- net N$12: now also D7.C; no longer D2.C
- net N$14: now also C13.1, D10.A, Q4.G, R25.1, R26.2; no longer C6.1, D5.A, R19.1, R7.2, T2.G
- net N$16: now also C10.1, R15.2; no longer C5.1, R30.2
- net N$17: now also Q3.B, R20.1, R21.1; no longer Q4.B, R17.1, R18.1
- net N$18: now also D11.A, R26.1; no longer D7.A, R7.1
- net N$19: now also C14.2, Q4.D; no longer C8.2, T2.D
- net N$2: now also C5.+, C6.1, Q1.D; no longer C10.+, C3.1, T1.D
- net N$20: now also D12.A; no longer D8.A
- net N$22: now also D8.A, R16.1, R17.2; no longer D10.A, R3.1, R6.2
- net N$24: now also Q5.G, R27.1, R28.1; no longer Q2.G, R20.1, R21.1
- net N$25: now also Q5.D; no longer Q2.D
- net N$27: now also R29.1, R30.1; no longer R22.1, R23.1
- net N$29: now also D2.A, R1.1; no longer D9.A, R24.1
- net N$3: now also C5.-, C6.2, D5.A; no longer C10.-, C3.2, D4.A
- net N$30: now also R4.1, R5.2, T1.C; no longer R29.1, R8.2, U$3.C
- net N$31: now also D2.C, R6.2, T1.B; no longer D9.C, R26.2, U$3.B
- net N$32: now also D3.C, R5.1, T2.B; no longer D11.C, R8.1, U$2.B
- net N$38: now also D3.A, R2.1; no longer D11.A, R25.1
- net N$4: now also R14.2; no longer R9.2
- net N$41: now also D4.A; no longer D12.A
- net N$46: now also C12.2, R22.2; no longer C9.2, R15.2
- net N$47: now also C12.1, R24.2; no longer C9.1, R31.2
- net N$6: now also D4.C, D8.C; no longer D10.C, D12.C
- net N$7: now also D9.A, Q2.G, R17.1; no longer D6.A, Q1.G, R6.1
- net N$9: now also D11.C, D12.C, Q3.C; no longer D7.C, D8.C, Q4.C
- net OUT+SENSED: now also R23.2, R24.1; no longer R14.2, R31.1
- net OUTPUT_TO_SENSE: now also C8.+, C9.1, D5.C, D6.C, R12.1; no longer C11.+, C4.1, D3.C, D4.C, R16.1
- net VIN: now also F1.2A, F1.2B, R8.2; no longer F2.2A, F2.2B, R1.2
Other:
- moved on the sheet: C12, C13, C14, C3, C4, C6, C7, C9, D11, D12, D2, D7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

Commit message: Fixed values and types of few parts
Parts:
- Q5: value IRL530 -> IRL530N
- Q6: value IRF530 -> IRL530N
- R14: value 47k -> 100k
- R18: value 15k -> 33k
- R19: value 4k7 -> 10k
- R26: value 220R -> 2k2
Changed lines of the file:
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@@
 <part name="B1" library="rectifier" deviceset="RB1A" device="" value="1.5A"/>
 <part name="D5" library="diode" deviceset="1N5908" device="" value="SB360"/>
-<part name="R18" library="rcl" deviceset="R-EU_" device="M0805" value="15k"/>
-<part name="R19" library="rcl" deviceset="R-EU_" device="M0805" value="4k7"/>
+<part name="R18" library="rcl" deviceset="R-EU_" device="M0805" value="33k"/>
+<part name="R19" library="rcl" deviceset="R-EU_" device="M0805" value="10k"/>
 <part name="C11" library="rcl" deviceset="C-EU" device="C0805" value="10n"/>
 <part name="AC_IN" library="con-wago-500" deviceset="W237-102" device=""/>
@@
 <part name="F1" library="fuse" deviceset="SHK20L" device="" value="F3.15A"/>
 <part name="Q2" library="triakcz" deviceset="BSS84" device=""/>
-<part name="R14" library="rcl" deviceset="R-EU_" device="M0805" value="47k"/>
+<part name="R14" library="rcl" deviceset="R-EU_" device="M0805" value="100k"/>
 <part name="X3" library="con-wago-500" deviceset="W237-102" device=""/>
 <part name="DC_IN" library="con-wago-500" deviceset="W237-102" device=""/>
@@
 <part name="R21" library="rcl" deviceset="R-EU_" device="M0805" value="100k"/>
 <part name="D10" library="diode" deviceset="ZENER-DIODE" device="SOD80C" value="BZV55C15SMD"/>
-<part name="R26" library="rcl" deviceset="R-EU_" device="M0805" value="220R"/>
+<part name="R26" library="rcl" deviceset="R-EU_" device="M0805" value="2k2"/>
 <part name="R25" library="rcl" deviceset="R-EU_" device="M0805" value="330k"/>
 <part name="C13" library="rcl" deviceset="C-EU" device="C0805" value="100n"/>
@@
 <part name="C4" library="rcl" deviceset="C-EU" device="C0805" value="10n"/>
 <part name="C3" library="rcl" deviceset="C-EU" device="C0805" value="1uF/50V"/>
-<part name="Q5" library="transistor-power" deviceset="IRF530" device="" value="IRL530"/>
-<part name="Q6" library="transistor-power" deviceset="IRF530" device="" value="IRF530"/>
+<part name="Q5" library="transistor-power" deviceset="IRF530" device="" value="IRL530N"/>
+<part name="Q6" library="transistor-power" deviceset="IRF530" device="" value="IRL530N"/>
 <part name="JP1" library="pinhead" deviceset="PINHD-1X2" device=""/>
 <part name="T2" library="triakcz" deviceset="BCV47" device=""/>
