File: hw/PowerExtractor.sch (EAGLE design)
At the start: 86 parts, among them IC1 LM358D, Q1 IRL530N, Q2 BSS84, Q3 BC847SMD, Q4 IRF7416, Q5 IRL530N, Q6 IRL530N, T1 BCV47, T2 BCV47, T3 BCV47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

Commit message: multiple fixes
Parts:
- removed D12: 1N4148MINIMELF, triakcz:1N4148MINIMELF
Connections:
- removed net N$20: D12.A, X4.PWM
- net ARDUINO_MAIN_LIGHT_CTRL: now also X4.PWM
- net N$9: no longer D12.C
Changed lines of the file:
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@@
 <part name="D11" library="triakcz" deviceset="1N4148" device="MINIMELF"/>
 <part name="X4" library="triakcz" deviceset="LDD700L" device=""/>
-<part name="D12" library="triakcz" deviceset="1N4148" device="MINIMELF"/>
 <part name="X5" library="con-wago-500" deviceset="W237-102" device=""/>
 <part name="C14" library="rcl" deviceset="C-EU" device="C0805" value="100n"/>
@@
 <instance part="D11" gate="G$1" x="500.38" y="48.26" rot="R270"/>
 <instance part="X4" gate="A" x="528.32" y="38.1"/>
-<instance part="D12" gate="G$1" x="513.08" y="43.18" rot="R180"/>
 <instance part="X5" gate="-1" x="556.26" y="40.64" rot="R180"/>
 <instance part="X5" gate="-2" x="556.26" y="45.72" rot="R180"/>
@@
 <segment>
 <pinref part="R20" gate="G$1" pin="2"/>
-<wire x1="312.42" y1="48.26" x2="312.42" y2="210.82" width="0.1524" layer="91"/>
+<wire x1="312.42" y1="48.26" x2="312.42" y2="53.34" width="0.1524" layer="91"/>
 <label x="312.42" y="185.42" size="1.778" layer="95" rot="R270"/>
+<wire x1="312.42" y1="53.34" x2="312.42" y2="210.82" width="0.1524" layer="91"/>
 <wire x1="312.42" y1="210.82" x2="114.3" y2="210.82" width="0.1524" layer="91"/>
 <pinref part="A1" gate="G$1" pin="D5"/>
+<pinref part="X4" gate="A" pin="PWM"/>
+<wire x1="525.78" y1="43.18" x2="322.58" y2="43.18" width="0.1524" layer="91"/>
+<wire x1="322.58" y1="43.18" x2="322.58" y2="53.34" width="0.1524" layer="91"/>
+<wire x1="322.58" y1="53.34" x2="312.42" y2="53.34" width="0.1524" layer="91"/>
+<junction x="312.42" y="53.34"/>
 </segment>
 </net>
@@
 <pinref part="Q3" gate="G$1" pin="C"/>
 <pinref part="D11" gate="G$1" pin="C"/>
-<wire x1="500.38" y1="45.72" x2="500.38" y2="43.18" width="0.1524" layer="91"/>
-<wire x1="500.38" y1="43.18" x2="500.38" y2="40.64" width="0.1524" layer="91"/>
-<junction x="500.38" y="43.18"/>
-<wire x1="500.38" y1="43.18" x2="510.54" y2="43.18" width="0.1524" layer="91"/>
-<pinref part="D12" gate="G$1" pin="C"/>
+<wire x1="500.38" y1="45.72" x2="500.38" y2="40.64" width="0.1524" layer="91"/>
 </segment>
 </net>
@@
 </segment>
 </net>
-<net name="N$20" class="0">
-<segment>
-<pinref part="X4" gate="A" pin="PWM"/>
-<pinref part="D12" gate="G$1" pin="A"/>
-<wire x1="515.62" y1="43.18" x2="525.78" y2="43.18" width="0.1524" layer="91"/>
-</segment>
-</net>
