File: hw/PowerExtractor.brd (EAGLE design)
At the start: 74.6 x 78.7 mm, 86 parts, among them IC1 LM358D, Q1 IRL530N, Q2 BSS84, Q3 BC847SMD, Q4 IRF7416, Q5 IRL530N, Q6 IRL530N, T1 BCV47, T2 BCV47, T3 BCV47, U1 ZXCT1086E5TA, U2 ZXCT1086E5TA, X4 LDD700L

Commit message: Fixing various bugs
Parts:
- moved Q4 1.27 mm to (41.9, 68.6), turned to 180 degrees
Connections:
- net ARDUINO_VIN_ANALOG renamed ARDUINO_VIN_SENSE
- net N$11 renamed ARDUINO_IOUT_SENSE
- net N$34 renamed DISPLAY_SDA
- net N$35 renamed DISPLAY_SCL
- net +5V: now also DSPL.2; no longer DSPL.1
- net GND: now also DSPL.1; no longer DSPL.2
- net LIGHTVCC: now also Q4.1, Q4.2, Q4.3; no longer Q4.5, Q4.6, Q4.7, Q4.8
- net N$19: now also Q4.5, Q4.6, Q4.7, Q4.8; no longer Q4.1, Q4.2, Q4.3
Routing:
- net GND: track 465.9 -> 433.0 mm
- net LIGHTVCC: track 55.6 -> 49.4 mm
- net N$19: track 47.2 -> 42.4 mm
- net N$14: track 14.3 -> 10.4 mm
- net +5V: track 86.6 -> 84.7 mm
Changed lines of the file:
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@@
 <layer number="48" name="Document" color="7" fill="1" visible="no" active="yes"/>
 <layer number="49" name="Reference" color="7" fill="1" visible="no" active="yes"/>
-<layer number="51" name="tDocu" color="7" fill="1" visible="no" active="yes"/>
-<layer number="52" name="bDocu" color="7" fill="1" visible="no" active="yes"/>
+<layer number="51" name="tDocu" color="7" fill="1" visible="yes" active="yes"/>
+<layer number="52" name="bDocu" color="7" fill="1" visible="yes" active="yes"/>
 <layer number="91" name="Nets" color="2" fill="1" visible="no" active="no"/>
 <layer number="92" name="Busses" color="1" fill="1" visible="no" active="no"/>
@@
 <attribute name="SUPPLIER" value="DIODES INC." x="-17.78" y="-11.43" size="1.778" layer="28" rot="MR0" display="off"/>
 </element>
-<element name="Q4" library="triakcz" package="SO-8" value="IRF7416" x="43.18" y="68.58" rot="MR270"/>
+<element name="Q4" library="triakcz" package="SO-8" value="IRF7416" x="41.91" y="68.58" rot="MR180"/>
 <element name="Q3" library="triakcz" package="SOT23" value="BC847SMD" x="67.31" y="63.5" rot="MR0"/>
 <element name="R20" library="rcl" package="0207/10" value="100k" x="63.5" y="44.45" rot="MR0"/>
@@
 <wire x1="19.685" y1="16.83" x2="18.1" y2="16.83" width="0.6096" layer="16"/>
 </signal>
-<signal name="ARDUINO_VIN_ANALOG">
+<signal name="ARDUINO_VIN_SENSE">
 <contactref element="R9" pad="2"/>
 <contactref element="R8" pad="1"/>
@@
 <contactref element="R30" pad="2"/>
 <contactref element="KEYBRD" pad="1"/>
-<contactref element="DSPL" pad="2"/>
 <contactref element="D1" pad="A"/>
 <contactref element="X3" pad="1"/>
@@
 <wire x1="12.7" y1="58.42" x2="15.24" y2="60.96" width="0.6096" layer="16"/>
 <wire x1="15.24" y1="60.96" x2="15.24" y2="63.4746" width="0.6096" layer="16"/>
-<wire x1="46.99" y1="63.5" x2="46.99" y2="58.42" width="0.6096" layer="1"/>
-<wire x1="46.99" y1="58.42" x2="50.8" y2="58.42" width="0.6096" layer="1"/>
-<wire x1="50.8" y1="58.42" x2="50.8" y2="46.99" width="0.6096" layer="1"/>
-<wire x1="50.8" y1="46.99" x2="41.91" y2="38.1" width="0.6096" layer="1"/>
 <contactref element="Q5" pad="S"/>
 <contactref element="Q6" pad="S"/>
@@
 <vertex x="0" y="2.54"/>
 </polygon>
+<contactref element="DSPL" pad="1"/>
 </signal>
 <signal name="ARDUINO_VOUT_SENSE">
@@
 </signal>
 <signal name="LIGHTVCC">
-<contactref element="Q4" pad="5"/>
-<contactref element="Q4" pad="6"/>
-<contactref element="Q4" pad="7"/>
-<contactref element="Q4" pad="8"/>
+<contactref element="Q4" pad="1"/>
+<contactref element="Q4" pad="2"/>
+<contactref element="Q4" pad="3"/>
 <contactref element="C13" pad="2"/>
 <contactref element="R25" pad="2"/>
@@
 <wire x1="23.114" y1="69.85" x2="18.034" y2="69.85" width="1.778" layer="1"/>
 <wire x1="44.41" y1="74.93" x2="44.41" y2="73.92" width="0.6096" layer="1"/>
-<wire x1="40.38" y1="70.485" x2="40.38" y2="70.9" width="1.4224" layer="16"/>
-<wire x1="40.38" y1="70.9" x2="40.62" y2="71.14" width="1.4224" layer="16"/>
 <wire x1="41.55" y1="72.07" x2="44.41" y2="74.93" width="1.4224" layer="16"/>
-<wire x1="40.38" y1="66.675" x2="40.38" y2="67.945" width="1.4224" layer="16"/>
-<wire x1="40.38" y1="67.945" x2="40.38" y2="69.215" width="1.4224" layer="16"/>
-<wire x1="40.38" y1="69.215" x2="40.38" y2="70.485" width="1.4224" layer="16"/>
 <wire x1="55.36" y1="72.07" x2="53.34" y2="72.07" width="0.6096" layer="16"/>
 <wire x1="50.8" y1="72.07" x2="41.55" y2="72.07" width="0.6096" layer="16"/>
 <wire x1="55.36" y1="72.07" x2="55.88" y2="72.185" width="0.6096" layer="16"/>
 <wire x1="53.34" y1="72.07" x2="50.8" y2="72.07" width="0.6096" layer="16"/>
-<wire x1="41.55" y1="72.07" x2="40.62" y2="71.14" width="1.4224" layer="16"/>
-<wire x1="40.62" y1="71.14" x2="40.64" y2="71.12" width="0.6096" layer="16"/>
-<wire x1="40.38" y1="70.9" x2="40.42" y2="70.9" width="1.4224" layer="16"/>
-<wire x1="40.42" y1="70.9" x2="40.64" y2="71.12" width="0.6096" layer="16"/>
+<wire x1="41.275" y1="71.38" x2="42.545" y2="71.38" width="0" layer="19" extent="16-16"/>
+<wire x1="40.005" y1="71.38" x2="41.275" y2="71.38" width="0" layer="19" extent="16-16"/>
+<wire x1="41.91" y1="69.85" x2="42.545" y2="71.38" width="0" layer="19" extent="1-16"/>
 </signal>
 <signal name="ARDUINO_VIN">
@@
 <wire x1="51.12" y1="69.85" x2="51.12" y2="67.945" width="0.6096" layer="16"/>
 <wire x1="51.12" y1="67.945" x2="49.85" y2="66.675" width="0.6096" layer="16"/>
-<wire x1="49.85" y1="66.675" x2="45.98" y2="66.675" width="0.6096" layer="16"/>
+<wire x1="43.815" y1="71.38" x2="49.85" y2="66.675" width="0" layer="19" extent="16-16"/>
 </signal>
 <signal name="N$17">
@@
 <signal name="N$19">
 <contactref element="X4" pad="VCC"/>
-<contactref element="Q4" pad="1"/>
-<contactref element="Q4" pad="2"/>
-<contactref element="Q4" pad="3"/>
+<contactref element="Q4" pad="5"/>
+<contactref element="Q4" pad="6"/>
+<contactref element="Q4" pad="7"/>
 <contactref element="C14" pad="2"/>
-<wire x1="45.98" y1="70.485" x2="45.98" y2="69.215" width="1.4224" layer="16"/>
-<wire x1="45.98" y1="67.945" x2="45.98" y2="69.215" width="0.6096" layer="16"/>
-<wire x1="45.98" y1="69.215" x2="48.26" y2="69.215" width="1.4224" layer="16"/>
 <via x="48.26" y="69.215" extent="1-16" drill="0.8" diameter="1.6764" shape="square"/>
 <wire x1="48.26" y1="69.215" x2="54.61" y2="69.215" width="1.4224" layer="1"/>
@@
 <wire x1="55.245" y1="69.53" x2="54.93" y2="69.215" width="0.6096" layer="1"/>
 <wire x1="54.93" y1="69.215" x2="54.61" y2="69.215" width="0.6096" layer="1"/>
+<contactref element="Q4" pad="8"/>
+<wire x1="42.545" y1="65.78" x2="43.815" y2="65.78" width="0" layer="19" extent="16-16"/>
+<wire x1="41.275" y1="65.78" x2="42.545" y2="65.78" width="0" layer="19" extent="16-16"/>
+<wire x1="40.005" y1="65.78" x2="41.275" y2="65.78" width="0" layer="19" extent="16-16"/>
+<wire x1="48.26" y1="69.215" x2="42.545" y2="65.78" width="0" layer="19" extent="16-16"/>
 </signal>
 <signal name="N$20">
@@
 <wire x1="44.45" y1="36.83" x2="44.45" y2="43.01" width="0.6096" layer="16"/>
 </signal>
-<signal name="N$34">
+<signal name="DISPLAY_SDA">
 <contactref element="DSPL" pad="4"/>
 <contactref element="A1" pad="A4"/>
 <wire x1="52.07" y1="63.5" x2="52.07" y2="52.07" width="0.6096" layer="16"/>
 </signal>
-<signal name="N$35">
+<signal name="DISPLAY_SCL">
 <contactref element="DSPL" pad="3"/>
 <contactref element="A1" pad="A5"/>
@@
 <wire x1="16.1798" y1="58.48" x2="18.415" y2="58.48" width="0.6096" layer="16"/>
 </signal>
-<signal name="N$11">
+<signal name="ARDUINO_IOUT_SENSE">
 <contactref element="IC1" pad="6"/>
 <contactref element="IC1" pad="7"/>
@@
 <contactref element="IC1" pad="8"/>
 <contactref element="A1" pad="5V"/>
-<contactref element="DSPL" pad="1"/>
 <wire x1="40.32" y1="48.895" x2="41.91" y2="50.485" width="0.6096" layer="16"/>
 <wire x1="41.91" y1="50.485" x2="41.91" y2="50.8" width="0.6096" layer="16"/>
@@
 <wire x1="40.32" y1="48.895" x2="41.91" y2="50.485" width="0.6096" layer="1"/>
 <wire x1="41.91" y1="50.485" x2="41.91" y2="52.07" width="0.6096" layer="1"/>
-<wire x1="48.26" y1="54.61" x2="48.26" y2="49.53" width="0.6096" layer="1"/>
+<wire x1="48.26" y1="55.88" x2="48.26" y2="49.53" width="0.6096" layer="1"/>
 <wire x1="48.26" y1="49.53" x2="46.99" y2="48.26" width="0.6096" layer="1"/>
 <wire x1="46.99" y1="48.26" x2="40.955" y2="48.26" width="0.6096" layer="1"/>
 <wire x1="40.955" y1="48.26" x2="40.32" y2="48.895" width="0.6096" layer="1"/>
-<wire x1="44.45" y1="63.5" x2="44.45" y2="58.42" width="0.6096" layer="1"/>
-<wire x1="44.45" y1="58.42" x2="47.625" y2="55.245" width="0.6096" layer="1"/>
-<wire x1="47.625" y1="55.245" x2="48.26" y2="54.61" width="0.6096" layer="1"/>
-<wire x1="48.26" y1="55.88" x2="47.625" y2="55.245" width="0.6096" layer="1"/>
 <wire x1="44.45" y1="49.21" x2="43.5" y2="49.21" width="0.6096" layer="16"/>
 <wire x1="43.5" y1="49.21" x2="42.545" y2="50.165" width="0.6096" layer="16"/>
 <wire x1="42.545" y1="49.21" x2="42.545" y2="50.165" width="0.6096" layer="16"/>
 <wire x1="42.545" y1="50.165" x2="41.91" y2="50.8" width="0.6096" layer="16"/>
+<contactref element="DSPL" pad="2"/>
+<wire x1="48.26" y1="55.88" x2="48.26" y2="60.96" width="0.6096" layer="1"/>
+<wire x1="48.26" y1="60.96" x2="46.99" y2="62.23" width="0.6096" layer="1"/>
+<wire x1="46.99" y1="62.23" x2="46.99" y2="63.5" width="0.6096" layer="1"/>
 </signal>
 <signal name="N$13">

Commit message: multiple fixes
Parts:
- removed D12: 1N4148MINIMELF, triakcz:SOD80C
Connections:
- removed net N$20: D12.A, X4.PWM
- net ARDUINO_MAIN_LIGHT_CTRL: now also X4.PWM
- net N$9: no longer D12.C
Routing:
- net N$20: track 2.74 -> 0.00 mm
- net N$9: track 9.09 -> 6.95 mm
Changed lines of the file:
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@@
 <element name="D11" library="triakcz" package="SOD80C" value="1N4148MINIMELF" x="57.15" y="66.04" rot="MR0"/>
 <element name="X4" library="triakcz" package="LDD_700L" value="LDD700L" x="67.31" y="55.88" rot="R90"/>
-<element name="D12" library="triakcz" package="SOD80C" value="1N4148MINIMELF" x="64.135" y="62.865" rot="MR270"/>
 <element name="X5" library="con-wago-500" package="W237-102" value="" x="52.07" y="76.2">
 <attribute name="OC_NEWARK" value="70K9898" x="149.86" y="12.7" size="1.778" layer="27" display="off"/>
@@
 <wire x1="58.42" y1="44.45" x2="52.07" y2="38.1" width="0.6096" layer="16"/>
 <wire x1="52.07" y1="38.1" x2="52.07" y2="36.83" width="0.6096" layer="16"/>
+<contactref element="X4" pad="PWM"/>
+<wire x1="58.42" y1="44.45" x2="64.135" y2="58.42" width="0" layer="19" extent="1-1"/>
 </signal>
 <signal name="N$9">
 <contactref element="Q3" pad="3"/>
 <contactref element="D11" pad="C"/>
-<contactref element="D12" pad="C"/>
-<wire x1="64.135" y1="64.565" x2="64.17" y2="64.6" width="0.6096" layer="16"/>
 <wire x1="64.17" y1="64.6" x2="67.31" y2="64.6" width="0.6096" layer="16"/>
-<wire x1="64.135" y1="64.565" x2="62.66" y2="66.04" width="0.6096" layer="16"/>
 <wire x1="62.66" y1="66.04" x2="58.85" y2="66.04" width="0.6096" layer="16"/>
+<wire x1="62.66" y1="66.04" x2="64.17" y2="64.6" width="0" layer="19" extent="16-16"/>
 </signal>
 <signal name="N$18">
@@
 <wire x1="48.26" y1="69.215" x2="42.545" y2="65.78" width="0" layer="19" extent="16-16"/>
 </signal>
-<signal name="N$20">
-<contactref element="X4" pad="PWM"/>
-<contactref element="D12" pad="A"/>
-<wire x1="64.135" y1="58.42" x2="64.135" y2="61.165" width="0.6096" layer="16"/>
-</signal>
 <signal name="N$24">
